Commit message: //修改urdf模型

File: src/space_driver/config/urdf0/urdf0.urdf (robot description, URDF)
Before this commit: robot urdf0, 8 links, 7 joints
Joints:
- joint joint4: axis 0 0 1 -> 0 0 -1
- joint joint6: origin xyz=0 0.6115 0 rpy=-1.5708 1.5708 0 -> xyz=0 0.6115 0 rpy=-1.5708 -1.5708 0

File: src/space_driver/config/urdf0/urdf0modified.urdf (robot description, URDF)
Before this commit: robot urdf0, 8 links, 7 joints
Joints:
- joint joint6: origin xyz=0 0.6115 0 rpy=-1.5708 1.5708 0 -> xyz=0 0.6115 0 rpy=-1.5708 -1.5708 0
