Commit message: //添加rviz可视化

File: src/space_driver/config/urdf0/urdf0_base_4.urdf (robot description, URDF)
Before this commit: robot urdf0, 8 links, 7 joints
Links:
- link Link1: geometry collision mesh filename=package://urdf0/meshes/Link1.STL; visual mesh filename=package://urdf0/meshes/Link1.STL
- link Link2: geometry collision mesh filename=package://urdf0/meshes/Link2.STL; visual mesh filename=package://urdf0/meshes/Link2.STL
- link Link3: geometry collision mesh filename=package://urdf0/meshes/Link3.STL; visual mesh filename=package://urdf0/meshes/Link3.STL
- link Link4: geometry collision mesh filename=package://urdf0/meshes/Link4.STL; visual mesh filename=package://urdf0/meshes/Link4.STL
- link Link5: geometry collision mesh filename=package://urdf0/meshes/Link5.STL; visual mesh filename=package://urdf0/meshes/Link5.STL
- link Link6: geometry collision mesh filename=package://urdf0/meshes/Link6.STL; visual mesh filename=package://urdf0/meshes/Link6.STL
- link Link7: geometry collision mesh filename=package://urdf0/meshes/Link7.STL; visual mesh filename=package://urdf0/meshes/Link7.STL
- link base_link: geometry collision mesh filename=package://urdf0/meshes/base_link.STL; visual mesh filename=package://urdf0/meshes/base_link.STL
Joints:
- joint joint1: origin xyz=0 0 0.38932 rpy=3.1416 0 0 -> xyz=0 0 0 rpy=0 0 0
- joint joint2: origin xyz=0 0.6115 0 rpy=1.5708 0 0 -> xyz=0 0 0 rpy=0 0 0
- joint joint3: origin xyz=0 -5.0815 0 rpy=-1.5708 0 0 -> xyz=0 0 0 rpy=0 0 0
- joint joint4: origin xyz=0 0 0 rpy=1.5708 1.5708 0 -> xyz=0 0 0 rpy=0 0 0

File: src/space_driver/config/urdf0/urdf0_copy.urdf (robot description, URDF)
Before this commit: robot urdf0, 8 links, 7 joints
Links:
- link Link1: geometry collision mesh filename=package://urdf0/meshes/Link1.STL; visual mesh filename=package://urdf0/meshes/Link1.STL
- link Link2: geometry collision mesh filename=package://urdf0/meshes/Link2.STL; visual mesh filename=package://urdf0/meshes/Link2.STL
- link Link3: geometry collision mesh filename=package://urdf0/meshes/Link3.STL; visual mesh filename=package://urdf0/meshes/Link3.STL
- link Link4: geometry collision mesh filename=package://urdf0/meshes/Link4.STL; visual mesh filename=package://urdf0/meshes/Link4.STL
- link Link5: geometry collision mesh filename=package://urdf0/meshes/Link5.STL; visual mesh filename=package://urdf0/meshes/Link5.STL
- link Link6: geometry collision mesh filename=package://urdf0/meshes/Link6.STL; visual mesh filename=package://urdf0/meshes/Link6.STL
- link Link7: geometry collision mesh filename=package://urdf0/meshes/Link7.STL; visual mesh filename=package://urdf0/meshes/Link7.STL
- link base_link: geometry collision mesh filename=package://urdf0/meshes/base_link.STL; visual mesh filename=package://urdf0/meshes/base_link.STL
Joints:
- joint joint1: type continuous -> fixed
- joint joint3: type continuous -> fixed
- joint joint6: type continuous -> fixed

File: src/space_driver/config/urdf0/urdf0fixed.urdf (robot description, URDF)
Before this commit: robot urdf0, 8 links, 7 joints
Joints:
- joint joint1: type continuous -> fixed
- joint joint3: type continuous -> fixed
- joint joint6: type continuous -> fixed

File: src/space_driver/config/urdf1/urdf1.urdf (robot description, URDF)
Before this commit: robot urdf0, 8 links, 7 joints
Links:
- removed link link_1
- removed link link_2
- removed link link_3
- removed link link_4
- removed link link_5
- removed link link_6
- removed link link_7
- added link Link1, mass 55.7444455513424; collision mesh filename=package://space_driver/config/urdf1/meshes/Link1.STL; visual mesh filename=package://space_driver/config/urdf1/meshes/Link1.STL
- added link Link2, mass 63.019; collision mesh filename=package://space_driver/config/urdf1/meshes/Link2.STL; visual mesh filename=package://space_driver/config/urdf1/meshes/Link2.STL
- added link Link3, mass 226.93; collision mesh filename=package://space_driver/config/urdf1/meshes/Link3.STL; visual mesh filename=package://space_driver/config/urdf1/meshes/Link3.STL
- added link Link4, mass 212.87; collision mesh filename=package://space_driver/config/urdf1/meshes/Link4.STL; visual mesh filename=package://space_driver/config/urdf1/meshes/Link4.STL
- added link Link5, mass 63.019; collision mesh filename=package://space_driver/config/urdf1/meshes/Link5.STL; visual mesh filename=package://space_driver/config/urdf1/meshes/Link5.STL
- added link Link6, mass 55.744; collision mesh filename=package://space_driver/config/urdf1/meshes/Link6.STL; visual mesh filename=package://space_driver/config/urdf1/meshes/Link6.STL
- added link Link7, mass 5.0287; collision mesh filename=package://space_driver/config/urdf1/meshes/Link7.STL; visual mesh filename=package://space_driver/config/urdf1/meshes/Link7.STL
- link base_link: geometry collision mesh filename=package://space_driver/config/urdf1/meshes/base_link.STL; visual mesh filename=package://space_driver/config/urdf1/meshes/base_link.STL
Joints:
- joint joint1: child link_1 -> Link1
- joint joint2: child link_2 -> Link2; origin xyz=0 0.6115 0 rpy=1.5708 0 0 -> xyz=0 0.6115 0 rpy=1.5708 1.5708 0; parent link_1 -> Link1
- joint joint3: axis 0 0 -1 -> 0 0 1; child link_3 -> Link3; origin xyz=0 -5.0815 0 rpy=1.5708 0 0 -> xyz=0 0 0 rpy=1.5708 0 0; parent link_2 -> Link2
- joint joint4: child link_4 -> Link4; origin xyz=0 0 0 rpy=1.5708 -1.5708 0 -> xyz=4.44 0 -0.035 rpy=-3.1416 0 1.5708; parent link_3 -> Link3
- joint joint5: child link_5 -> Link5; origin xyz=4.44 0 0.035 rpy=0 0 -1.5708 -> xyz=0 5.0815 0 rpy=-1.5708 0 0; parent link_4 -> Link4
- joint joint6: child link_6 -> Link6; origin xyz=0 0.6115 0 rpy=-1.5708 -1.5708 0 -> xyz=0 -0.6115 0 rpy=1.5708 0 0; parent link_5 -> Link5
- joint joint7: child link_7 -> Link7; origin xyz=0 -0.3645 0 rpy=1.5708 0 0 -> xyz=0 0.38932 0 rpy=-1.5708 0 0; parent link_6 -> Link6

File: src/space_driver/config/urdf1/urdf1fixed.urdf (robot description, URDF)
Before this commit: robot urdf0, 8 links, 7 joints
Links:
- link Link1: mass 55.744 -> 55.7444455513424; geometry collision mesh filename=package://space_driver/config/urdf1/meshes/Link1.STL; visual mesh filename=package://space_driver/config/urdf1/meshes/Link1.STL
- link Link2: geometry collision mesh filename=package://space_driver/config/urdf1/meshes/Link2.STL; visual mesh filename=package://space_driver/config/urdf1/meshes/Link2.STL
- link Link3: mass 212.87 -> 226.93; geometry collision mesh filename=package://space_driver/config/urdf1/meshes/Link3.STL; visual mesh filename=package://space_driver/config/urdf1/meshes/Link3.STL
- link Link4: mass 226.93 -> 212.87; geometry collision mesh filename=package://space_driver/config/urdf1/meshes/Link4.STL; visual mesh filename=package://space_driver/config/urdf1/meshes/Link4.STL
- link Link5: geometry collision mesh filename=package://space_driver/config/urdf1/meshes/Link5.STL; visual mesh filename=package://space_driver/config/urdf1/meshes/Link5.STL
- link Link6: geometry collision mesh filename=package://space_driver/config/urdf1/meshes/Link6.STL; visual mesh filename=package://space_driver/config/urdf1/meshes/Link6.STL
- link Link7: geometry collision mesh filename=package://space_driver/config/urdf1/meshes/Link7.STL; visual mesh filename=package://space_driver/config/urdf1/meshes/Link7.STL
- link base_link: geometry collision mesh filename=package://space_driver/config/urdf1/meshes/base_link.STL; visual mesh filename=package://space_driver/config/urdf1/meshes/base_link.STL
Joints:
- joint joint1: origin xyz=0 0 0.38932 rpy=3.1416 0 0 -> xyz=0 0 0.3645 rpy=3.1416 0 0; type continuous -> fixed
- joint joint2: origin xyz=0 0.6115 0 rpy=1.5708 0 0 -> xyz=0 0.6115 0 rpy=1.5708 1.5708 0; type continuous -> fixed
- joint joint3: origin xyz=0 -5.0815 0 rpy=-1.5708 0 0 -> xyz=0 0 0 rpy=1.5708 0 0
- joint joint4: origin xyz=0 0 0 rpy=1.5708 1.5708 0 -> xyz=4.44 0 -0.035 rpy=-3.1416 0 1.5708
- joint joint5: origin xyz=4.44 0 -0.035 rpy=3.1416 0 0 -> xyz=0 5.0815 0 rpy=-1.5708 0 0; type continuous -> fixed
- joint joint6: origin xyz=0 -0.6115 0 rpy=1.5708 1.5708 0 -> xyz=0 -0.6115 0 rpy=1.5708 0 0
- joint joint7: origin xyz=0 0.3645 0 rpy=-1.5708 0 0 -> xyz=0 0.38932 0 rpy=-1.5708 0 0

File: src/space_driver/config/urdf_prv/urdf0.urdf (robot description, URDF)
Before this commit: robot urdf0, 8 links, 7 joints
Links:
- removed link Link1
- removed link Link2
- removed link Link3
- removed link Link4
- removed link Link5
- removed link Link6
- removed link Link7
- added link link_1, mass 55.7444455513422; collision mesh filename=package://urdf0/meshes/Link1.STL; visual mesh filename=package://urdf0/meshes/Link1.STL
- added link link_2, mass 63.0188095750657; collision mesh filename=package://urdf0/meshes/Link2.STL; visual mesh filename=package://urdf0/meshes/Link2.STL
- added link link_3, mass 212.870919787655; collision mesh filename=package://urdf0/meshes/Link3.STL; visual mesh filename=package://urdf0/meshes/Link3.STL
- added link link_4, mass 226.927653025662; collision mesh filename=package://urdf0/meshes/Link4.STL; visual mesh filename=package://urdf0/meshes/Link4.STL
- added link link_5, mass 63.0188095750638; collision mesh filename=package://urdf0/meshes/Link5.STL; visual mesh filename=package://urdf0/meshes/Link5.STL
- added link link_6, mass 55.7444455513433; collision mesh filename=package://urdf0/meshes/Link6.STL; visual mesh filename=package://urdf0/meshes/Link6.STL
- added link link_7, mass 5.02870680905465; collision mesh filename=package://urdf0/meshes/Link7.STL; visual mesh filename=package://urdf0/meshes/Link7.STL
- link base_link: geometry collision mesh filename=package://urdf0/meshes/base_link.STL; visual mesh filename=package://urdf0/meshes/base_link.STL
Joints:
- joint joint1: child Link1 -> link_1; origin xyz=0 0 0.38932 rpy=3.1416 0 0 -> xyz=0 0 0.3645 rpy=3.1416 0 0
- joint joint2: child Link2 -> link_2; parent Link1 -> link_1
- joint joint3: axis 0 0 1 -> 0 0 -1; child Link3 -> link_3; origin xyz=0 -5.0815 0 rpy=-1.5708 0 0 -> xyz=0 -5.0815 0 rpy=1.5708 0 0; parent Link2 -> link_2
- joint joint4: axis 0 0 1 -> 0 0 -1; child Link4 -> link_4; origin xyz=0 0 0 rpy=1.5708 1.5708 0 -> xyz=0 0 0 rpy=1.5708 -1.5708 0; parent Link3 -> link_3
- joint joint5: child Link5 -> link_5; origin xyz=4.44 0 -0.035 rpy=3.1416 0 0 -> xyz=4.44 0 0.035 rpy=0 0 -3.1415926535; parent Link4 -> link_4
- joint joint6: child Link6 -> link_6; origin xyz=0 -0.6115 0 rpy=1.5708 1.5708 0 -> xyz=0 0.6115 0 rpy=-1.5708 -1.5708 0; parent Link5 -> link_5
- joint joint7: child Link7 -> link_7; origin xyz=0 0.3645 0 rpy=-1.5708 0 0 -> xyz=0 -0.3645 0 rpy=1.5708 0 0; parent Link6 -> link_6

File: src/space_driver/config/urdf_prv/urdf0modified.urdf (robot description, URDF)
Before this commit: robot urdf0, 8 links, 7 joints
Links:
- removed link Link1
- removed link Link2
- removed link Link3
- removed link Link4
- removed link Link5
- removed link Link6
- removed link Link7
- added link link_1, mass 55.7444455513422; collision mesh filename=package://urdf0/meshes/Link1.STL; visual mesh filename=package://urdf0/meshes/Link1.STL
- added link link_2, mass 63.0188095750657; collision mesh filename=package://urdf0/meshes/Link2.STL; visual mesh filename=package://urdf0/meshes/Link2.STL
- added link link_3, mass 212.870919787655; collision mesh filename=package://urdf0/meshes/Link3.STL; visual mesh filename=package://urdf0/meshes/Link3.STL
- added link link_4, mass 226.927653025662; collision mesh filename=package://urdf0/meshes/Link4.STL; visual mesh filename=package://urdf0/meshes/Link4.STL
- added link link_5, mass 63.0188095750638; collision mesh filename=package://urdf0/meshes/Link5.STL; visual mesh filename=package://urdf0/meshes/Link5.STL
- added link link_6, mass 55.7444455513433; collision mesh filename=package://urdf0/meshes/Link6.STL; visual mesh filename=package://urdf0/meshes/Link6.STL
- added link link_7, mass 5.02870680905465; collision mesh filename=package://urdf0/meshes/Link7.STL; visual mesh filename=package://urdf0/meshes/Link7.STL
- link base_link: geometry collision mesh filename=package://urdf0/meshes/base_link.STL; visual mesh filename=package://urdf0/meshes/base_link.STL
Joints:
- joint joint1: child Link1 -> link_1; origin xyz=0 0 0.38932 rpy=3.1416 0 0 -> xyz=0 0 0.3645 rpy=3.1416 0 0
- joint joint2: child Link2 -> link_2; parent Link1 -> link_1
- joint joint3: axis 0 0 1 -> 0 0 -1; child Link3 -> link_3; origin xyz=0 -5.0815 0 rpy=-1.5708 0 0 -> xyz=0 -5.0815 0 rpy=1.5708 0 0; parent Link2 -> link_2
- joint joint4: axis 0 0 1 -> 0 0 -1; child Link4 -> link_4; origin xyz=0 0 0 rpy=1.5708 1.5708 0 -> xyz=0 0 0 rpy=1.5708 -1.5708 0; parent Link3 -> link_3
- joint joint5: child Link5 -> link_5; origin xyz=4.44 0 -0.035 rpy=3.1416 0 0 -> xyz=4.44 0 0.035 rpy=0 0 -3.1415926535; parent Link4 -> link_4
- joint joint6: child Link6 -> link_6; origin xyz=0 -0.6115 0 rpy=1.5708 1.5708 0 -> xyz=0 0.6115 0 rpy=-1.5708 -1.5708 0; parent Link5 -> link_5
- joint joint7: child Link7 -> link_7; origin xyz=0 0.3645 0 rpy=-1.5708 0 0 -> xyz=0 -0.3645 0 rpy=1.5708 0 0; parent Link6 -> link_6
